Commit message: Modified camera settings

File: arm_description/urdf/arm_camera.xacro (robot description, xacro)
@@ -12,5 +12,5 @@
         <parent link="${camera_parent_link}"/>
         <child link="${camera_name}_link"/>
-        <origin xyz="0 0 0.00" rpy="0.0 1.57 0"/>
+        <origin xyz="0 0 0.00" rpy="0.0 0.30 0"/>
     </joint>
   <gazebo>
@@ -29,5 +29,5 @@
       </image>
       <clip>
-        <near>0.1</near>
+        <near>0.05</near>
         <far>100</far>
       </clip>
