Commit message: Modified mesh path

File: arm_description/urdf/arm.urdf.xacro (robot description, xacro)
@@ -13,5 +13,5 @@
     <visual>
       <geometry>
-        <mesh filename="package://arm_description/meshes/base_link.stl" scale="0.001 0.001 0.001"/>
+        <mesh filename="file://$(find arm_description)/meshes/base_link.stl" scale="0.001 0.001 0.001"/>
       </geometry>
       <origin rpy="0 0 0" xyz="0 0 0"/>
